File: KiCad/ISA8_Ethernet.kicad_pcb (KiCad board)
At the start: 2 copper layers, 104.1 x 74.9 mm, 34 parts, among them J1 RJMG1BD3B8K1ANR, J2 MEM_EXT, SW1 CONFIG, SW2 IRQ, SW3 IO_ADDR, SW4 ROM_ADDR, U1 RTL8019AS, U2 SST39SF040, U3 93LC46C, Y1 20MHz

Commit message: Update KiCad files
Signed-off-by: Sergey Kiselev <skiselev@gmail.com>
Parts:
- C10, C9: footprint Capacitor_Tantalum_SMD:CP_EIA-2012-15_AVX-P_Pad1.30x1.05mm_HandSolder -> Capacitor_Tantalum_SMD:CP_EIA-3528-15_AVX-H_Pad1.50x2.35mm_HandSolder
- moved C10 0.32 mm to (106.7, 119.1)
- moved C9 0.32 mm to (165.1, 119.1)
Routing:
- net GND: track 520.9 -> 538.4 mm
- net VCC: track 419.6 -> 426.0 mm
- net /IOCHRDY: track 43.0 -> 44.2 mm
- net /AEN: track 43.5 -> 44.4 mm
- net /~SMEMW: track 128.8 -> 129.6 mm
- net /~SMEMR: track 114.2 -> 114.7 mm
