File: KiCad/ISA8_Ethernet.sch (KiCad schematic (older format))
At the start: 32 parts, among them J1 RJMG1BD3B8K1ANR, J2 MEM_EXT, SW1 CONFIG, SW2 IRQ, SW3 IO_ADDR, SW4 ROM_ADDR, U1 RTL8019AS, U2 SST39SF040, U3 93LC46C, Y1 20MHz

Commit message: Update KiCad files
Signed-off-by: Sergey Kiselev <skiselev@gmail.com>
Parts:
- C10, C9: footprint Capacitor_Tantalum_SMD:CP_EIA-2012-15_AVX-P_Pad1.30x1.05mm_HandSolder -> Capacitor_Tantalum_SMD:CP_EIA-3528-15_AVX-H_Pad1.50x2.35mm_HandSolder
Changed lines of the file:
@@
 F 0 "C9" H 1925 7250 50  0000 L CNN
 F 1 "22uF" H 1925 7050 50  0000 L CNN
-F 2 "Capacitor_Tantalum_SMD:CP_EIA-2012-15_AVX-P_Pad1.30x1.05mm_HandSolder" H 1900 7150 50  0001 C CNN
+F 2 "Capacitor_Tantalum_SMD:CP_EIA-3528-15_AVX-H_Pad1.50x2.35mm_HandSolder" H 1900 7150 50  0001 C CNN
 F 3 "" H 1900 7150 50  0000 C CNN
 	1    1900 7150
@@
 F 0 "C10" H 2225 7250 50  0000 L CNN
 F 1 "22uF" H 2225 7050 50  0000 L CNN
-F 2 "Capacitor_Tantalum_SMD:CP_EIA-2012-15_AVX-P_Pad1.30x1.05mm_HandSolder" H 2200 7150 50  0001 C CNN
+F 2 "Capacitor_Tantalum_SMD:CP_EIA-3528-15_AVX-H_Pad1.50x2.35mm_HandSolder" H 2200 7150 50  0001 C CNN
 F 3 "" H 2200 7150 50  0000 C CNN
 	1    2200 7150
